File: schematic/EE1111A/EE1111A.kicad_sch (KiCad schematic)
At the start: 20 parts, among them J1 Power, J2 Digital/PWM, J3 Analog, J4 Digital/PWM, M1 Motor_Servo, Q1 2N2222, Q2 PN2907A, Q3 IRF9530, U1 INA219AxD

Commit message: Simulation Verified Schematic
Parts:
- L1: value 33uH -> 150uH
Changed lines of the file:
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@@
 			)
 		)
-		(property "Value" "33uH"
+		(property "Value" "150uH"
 			(at 177.8 137.16 90)
 			(show_name no)
