File: schematic/EE1111A.kicad_sch (KiCad schematic)
At the start: 20 parts, among them J1 Power, J2 Digital/PWM, J3 Analog, J4 Digital/PWM, M1 Motor_Servo, Q1 2N2222, Q2 PN2907A, Q3 IRF9530, U1 INA219AxD

Commit message: Fixed Errors
Parts:
- added Q6: 2N2222, symbol Simulation_SPICE:NPN
- added R13: 4.7k, symbol Device:R
Connections:
- net GND: now also Q6.3 (E)
- net at C1.1, D1.1 (K), Q1.1 (C)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: now also R13.2
- net at Q1.2 (B), Q2.2 (B): now also Q6.1 (C), R13.1; no longer R3.1
- new net: Q6.2 (B), R3.1
Other:
- moved on the sheet: R3
